File: hardware/nordic_tag/nRF52811.sch (KiCad schematic (older format))
At the start: 17 parts

Commit message: Started PCB + BOM
Parts:
- C201, C202, C203, C204, C205, C206, C207, C208, C209: renamed from C?; footprint (none) -> Capacitor_SMD:C_0603_1608Metric
- D201, D202: renamed from D?; footprint (none) -> LED_SMD:LED_0603_1608Metric
- R201, R202, R203: renamed from R?; footprint (none) -> Resistor_SMD:R_0603_1608Metric
- SW201: renamed from SW?; footprint (none) -> Button_Switch_SMD:SW_Push_1P1T_NO_CK_KMR2
- Y201: renamed from Y?; footprint (none) -> Crystal:Crystal_SMD_5032-2Pin_5.0x3.2mm_HandSoldering
- gave numbers to parts that had none: 1
Changed lines of the file:
@@
 EESchema Schematic File Version 4
+LIBS:nordic_tag-cache
 EELAYER 30 0
 EELAYER END
@@
 P 5650 3750
 AR Path="/5DCD44A3" Ref="U?"  Part="1"
-AR Path="/5DCA970B/5DCD44A3" Ref="U?"  Part="1"
-F 0 "U?" H 5675 2511 50  0000 C CNN
+AR Path="/5DCA970B/5DCD44A3" Ref="U201"  Part="1"
+F 0 "U201" H 5675 2511 50  0000 C CNN
 F 1 "nRF52811-QCAA" H 5675 2420 50  0000 C CNN
 F 2 "Package_DFN_QFN:QFN-32-1EP_5x5mm_P0.5mm_EP3.6x3.6mm" H 5600 2100 50  0001 C CNN
@@
 P 5450 5300
 AR Path="/5DCD44AE" Ref="#PWR?"  Part="1"
-AR Path="/5DCA970B/5DCD44AE" Ref="#PWR?"  Part="1"
-F 0 "#PWR?" H 5450 5050 50  0001 C CNN
+AR Path="/5DCA970B/5DCD44AE" Ref="#PWR0206"  Part="1"
+F 0 "#PWR0206" H 5450 5050 50  0001 C CNN
 F 1 "GND" H 5455 5127 50  0000 C CNN
 F 2 "" H 5450 5300 50  0001 C CNN
@@
 P 5150 2450
 AR Path="/5DCD44B9" Ref="#PWR?"  Part="1"
-AR Path="/5DCA970B/5DCD44B9" Ref="#PWR?"  Part="1"
-F 0 "#PWR?" H 5150 2300 50  0001 C CNN
+AR Path="/5DCA970B/5DCD44B9" Ref="#PWR0205"  Part="1"
+F 0 "#PWR0205" H 5150 2300 50  0001 C CNN
 F 1 "+3V3" H 5165 2623 50  0000 C CNN
 F 2 "" H 5150 2450 50  0001 C CNN
@@
 P 3200 3550
 AR Path="/5DCD44C4" Ref="R?"  Part="1"
-AR Path="/5DCA970B/5DCD44C4" Ref="R?"  Part="1"
-F 0 "R?" H 3270 3596 50  0000 L CNN
+AR Path="/5DCA970B/5DCD44C4" Ref="R201"  Part="1"
+F 0 "R201" H 3270 3596 50  0000 L CNN
 F 1 "10K" H 3270 3505 50  0000 L CNN
-F 2 "" V 3130 3550 50  0001 C CNN
+F 2 "Resistor_SMD:R_0603_1608Metric" V 3130 3550 50  0001 C CNN
 F 3 "~" H 3200 3550 50  0001 C CNN
 	1    3200 3550
@@
 P 3200 3200
 AR Path="/5DCD44CC" Ref="#PWR?"  Part="1"
-AR Path="/5DCA970B/5DCD44CC" Ref="#PWR?"  Part="1"
-F 0 "#PWR?" H 3200 3050 50  0001 C CNN
+AR Path="/5DCA970B/5DCD44CC" Ref="#PWR0202"  Part="1"
+F 0 "#PWR0202" H 3200 3050 50  0001 C CNN
 F 1 "+3V3" H 3215 3373 50  0000 C CNN
 F 2 "" H 3200 3200 50  0001 C CNN
@@
 P 2950 3850
 AR Path="/5DCD44D5" Ref="SW?"  Part="1"
-AR Path="/5DCA970B/5DCD44D5" Ref="SW?"  Part="1"
-F 0 "SW?" H 2950 4135 50  0000 C CNN
+AR Path="/5DCA970B/5DCD44D5" Ref="SW201"  Part="1"
+F 0 "SW201" H 2950 4135 50  0000 C CNN
 F 1 "SW_Push" H 2950 4044 50  0000 C CNN
-F 2 "" H 2950 4050 50  0001 C CNN
+F 2 "Button_Switch_SMD:SW_Push_1P1T_NO_CK_KMR2" H 2950 4050 50  0001 C CNN
 F 3 "~" H 2950 4050 50  0001 C CNN
 	1    2950 3850
@@
 P 2600 3950
 AR Path="/5DCD44DD" Ref="#PWR?"  Part="1"
-AR Path="/5DCA970B/5DCD44DD" Ref="#PWR?"  Part="1"
-F 0 "#PWR?" H 2600 3700 50  0001 C CNN
+AR Path="/5DCA970B/5DCD44DD" Ref="#PWR0201"  Part="1"
+F 0 "#PWR0201" H 2600 3700 50  0001 C CNN
 F 1 "GND" H 2605 3777 50  0000 C CNN
 F 2 "" H 2600 3950 50  0001 C CNN
@@
 P 4250 4450
 AR Path="/5DCD44E5" Ref="Y?"  Part="1"
-AR Path="/5DCA970B/5DCD44E5" Ref="Y?"  Part="1"
-F 0 "Y?" V 4204 4581 50  0000 L CNN
+AR Path="/5DCA970B/5DCD44E5" Ref="Y201"  Part="1"
+F 0 "Y201" V 4204 4581 50  0000 L CNN
 F 1 "32MHz" V 4295 4581 50  0000 L CNN
-F 2 "" H 4250 4450 50  0001 C CNN
+F 2 "Crystal:Crystal_SMD_5032-2Pin_5.0x3.2mm_HandSoldering" H 4250 4450 50  0001 C CNN
 F 3 "~" H 4250 4450 50  0001 C CNN
 	1    4250 4450
@@
 P 3900 4700
 AR Path="/5DCD44F1" Ref="C?"  Part="1"
-AR Path="/5DCA970B/5DCD44F1" Ref="C?"  Part="1"
-F 0 "C?" H 3992 4746 50  0000 L CNN
+AR Path="/5DCA970B/5DCD44F1" Ref="C202"  Part="1"
+F 0 "C202" H 3992 4746 50  0000 L CNN
 F 1 "12p" H 3992 4655 50  0000 L CNN
-F 2 "" H 3900 4700 50  0001 C CNN
+F 2 "Capacitor_SMD:C_0603_1608Metric" H 3900 4700 50  0001 C CNN
 F 3 "~" H 3900 4700 50  0001 C CNN
 	1    3900 4700
@@
 P 4250 4700
 AR Path="/5DCD44F7" Ref="C?"  Part="1"
-AR Path="/5DCA970B/5DCD44F7" Ref="C?"  Part="1"
-F 0 "C?" H 4342 4746 50  0000 L CNN
+AR Path="/5DCA970B/5DCD44F7" Ref="C204"  Part="1"
+F 0 "C204" H 4342 4746 50  0000 L CNN
 F 1 "12p" H 4342 4655 50  0000 L CNN
-F 2 "" H 4250 4700 50  0001 C CNN
+F 2 "Capacitor_SMD:C_0603_1608Metric" H 4250 4700 50  0001 C CNN
 F 3 "~" H 4250 4700 50  0001 C CNN
 	1    4250 4700
@@
 P 4250 4900
 AR Path="/5DCD4502" Ref="#PWR?"  Part="1"
-AR Path="/5DCA970B/5DCD4502" Ref="#PWR?"  Part="1"
-F 0 "#PWR?" H 4250 4650 50  0001 C CNN
+AR Path="/5DCA970B/5DCD4502" Ref="#PWR0204"  Part="1"
+F 0 "#PWR0204" H 4250 4650 50  0001 C CNN
 F 1 "GND" H 4255 4727 50  0000 C CNN
 F 2 "" H 4250 4900 50  0001 C CNN
@@
 P 5850 2350
 AR Path="/5DCD4508" Ref="C?"  Part="1"
-AR Path="/5DCA970B/5DCD4508" Ref="C?"  Part="1"
-F 0 "C?" H 5942 2396 50  0000 L CNN
+AR Path="/5DCA970B/5DCD4508" Ref="C206"  Part="1"
+F 0 "C206" H 5942 2396 50  0000 L CNN
 F 1 "1u" H 5942 2305 50  0000 L CNN
-F 2 "" H 5850 2350 50  0001 C CNN
+F 2 "Capacitor_SMD:C_0603_1608Metric" H 5850 2350 50  0001 C CNN
 F 3 "~" H 5850 2350 50  0001 C CNN
 	1    5850 2350
@@
 P 6250 2350
 AR Path="/5DCD450E" Ref="C?"  Part="1"
-AR Path="/5DCA970B/5DCD450E" Ref="C?"  Part="1"
-F 0 "C?" H 6342 2396 50  0000 L CNN
+AR Path="/5DCA970B/5DCD450E" Ref="C207"  Part="1"
+F 0 "C207" H 6342 2396 50  0000 L CNN
 F 1 "100p" H 6342 2305 50  0000 L CNN
-F 2 "" H 6250 2350 50  0001 C CNN
+F 2 "Capacitor_SMD:C_0603_1608Metric" H 6250 2350 50  0001 C CNN
 F 3 "~" H 6250 2350 50  0001 C CNN
 	1    6250 2350
@@
 P 6650 2350
 AR Path="/5DCD4514" Ref="C?"  Part="1"
-AR Path="/5DCA970B/5DCD4514" Ref="C?"  Part="1"
-F 0 "C?" H 6742 2396 50  0000 L CNN
+AR Path="/5DCA970B/5DCD4514" Ref="C208"  Part="1"
+F 0 "C208" H 6742 2396 50  0000 L CNN
 F 1 "NC" H 6742 2305 50  0000 L CNN
-F 2 "" H 6650 2350 50  0001 C CNN
+F 2 "Capacitor_SMD:C_0603_1608Metric" H 6650 2350 50  0001 C CNN
 F 3 "~" H 6650 2350 50  0001 C CNN
 	1    6650 2350
@@
 P 7050 2350
 AR Path="/5DCD451A" Ref="C?"  Part="1"
-AR Path="/5DCA970B/5DCD451A" Ref="C?"  Part="1"
-F 0 "C?" H 7142 2396 50  0000 L CNN
+AR Path="/5DCA970B/5DCD451A" Ref="C209"  Part="1"
+F 0 "C209" H 7142 2396 50  0000 L CNN
 F 1 "100n" H 7142 2305 50  0000 L CNN
-F 2 "" H 7050 2350 50  0001 C CNN
+F 2 "Capacitor_SMD:C_0603_1608Metric" H 7050 2350 50  0001 C CNN
 F 3 "~" H 7050 2350 50  0001 C CNN
 	1    7050 2350
@@
 P 7450 2450
 AR Path="/5DCD452D" Ref="#PWR?"  Part="1"
-AR Path="/5DCA970B/5DCD452D" Ref="#PWR?"  Part="1"
-F 0 "#PWR?" H 7450 2200 50  0001 C CNN
+AR Path="/5DCA970B/5DCD452D" Ref="#PWR0207"  Part="1"
+F 0 "#PWR0207" H 7450 2200 50  0001 C CNN
 F 1 "GND" H 7455 2277 50  0000 C CNN
 F 2 "" H 7450 2450 50  0001 C CNN
@@
 P 3700 2600
 AR Path="/5DCD453E" Ref="C?"  Part="1"
-AR Path="/5DCA970B/5DCD453E" Ref="C?"  Part="1"
-F 0 "C?" H 3792 2646 50  0000 L CNN
+AR Path="/5DCA970B/5DCD453E" Ref="C201"  Part="1"
+F 0 "C201" H 3792 2646 50  0000 L CNN
 F 1 "4u7" H 3792 2555 50  0000 L CNN
-F 2 "" H 3700 2600 50  0001 C CNN
+F 2 "Capacitor_SMD:C_0603_1608Metric" H 3700 2600 50  0001 C CNN
 F 3 "~" H 3700 2600 50  0001 C CNN
 	1    3700 2600
@@
 P 4050 2600
 AR Path="/5DCD4544" Ref="C?"  Part="1"
-AR Path="/5DCA970B/5DCD4544" Ref="C?"  Part="1"
-F 0 "C?" H 4142 2646 50  0000 L CNN
+AR Path="/5DCA970B/5DCD4544" Ref="C203"  Part="1"
+F 0 "C203" H 4142 2646 50  0000 L CNN
 F 1 "100n" H 4142 2555 50  0000 L CNN
-F 2 "" H 4050 2600 50  0001 C CNN
+F 2 "Capacitor_SMD:C_0603_1608Metric" H 4050 2600 50  0001 C CNN
 F 3 "~" H 4050 2600 50  0001 C CNN
 	1    4050 2600
@@
 P 4450 2600
 AR Path="/5DCD454A" Ref="C?"  Part="1"
-AR Path="/5DCA970B/5DCD454A" Ref="C?"  Part="1"
-F 0 "C?" H 4542 2646 50  0000 L CNN
+AR Path="/5DCA970B/5DCD454A" Ref="C205"  Part="1"
+F 0 "C205" H 4542 2646 50  0000 L CNN
 F 1 "100n" H 4542 2555 50  0000 L CNN
-F 2 "" H 4450 2600 50  0001 C CNN
+F 2 "Capacitor_SMD:C_0603_1608Metric" H 4450 2600 50  0001 C CNN
 F 3 "~" H 4450 2600 50  0001 C CNN
 	1    4450 2600
@@
 P 3700 2850
 AR Path="/5DCD455C" Ref="#PWR?"  Part="1"
-AR Path="/5DCA970B/5DCD455C" Ref="#PWR?"  Part="1"
-F 0 "#PWR?" H 3700 2600 50  0001 C CNN
+AR Path="/5DCA970B/5DCD455C" Ref="#PWR0203"  Part="1"
+F 0 "#PWR0203" H 3700 2600 50  0001 C CNN
 F 1 "GND" H 3705 2677 50  0000 C CNN
 F 2 "" H 3700 2850 50  0001 C CNN
@@
 LED1
 $Comp
-L Device:LED D?
+L Device:LED D201
 U 1 1 5DD8ABA8
 P 8500 5400
-F 0 "D?" V 8539 5283 50  0000 R CNN
+F 0 "D201" V 8539 5283 50  0000 R CNN
 F 1 "LED" V 8448 5283 50  0000 R CNN
-F 2 "" H 8500 5400 50  0001 C CNN
+F 2 "LED_SMD:LED_0603_1608Metric" H 8500 5400 50  0001 C CNN
 F 3 "~" H 8500 5400 50  0001 C CNN
 	1    8500 5400
@@
 $EndComp
 $Comp
-L Device:LED D?
+L Device:LED D202
 U 1 1 5DD8B03E
 P 8850 5400
-F 0 "D?" V 8889 5283 50  0000 R CNN
+F 0 "D202" V 8889 5283 50  0000 R CNN
 F 1 "LED" V 8798 5283 50  0000 R CNN
-F 2 "" H 8850 5400 50  0001 C CNN
+F 2 "LED_SMD:LED_0603_1608Metric" H 8850 5400 50  0001 C CNN
 F 3 "~" H 8850 5400 50  0001 C CNN
 	1    8850 5400
@@
 	8850 5550 8850 5700
 $Comp
-L Device:R R?
+L Device:R R202
 U 1 1 5DD8DC1B
 P 8500 5850
-F 0 "R?" H 8570 5896 50  0000 L CNN
+F 0 "R202" H 8570 5896 50  0000 L CNN
 F 1 "1k" H 8570 5805 50  0000 L CNN
-F 2 "" V 8430 5850 50  0001 C CNN
+F 2 "Resistor_SMD:R_0603_1608Metric" V 8430 5850 50  0001 C CNN
 F 3 "~" H 8500 5850 50  0001 C CNN
 	1    8500 5850
@@
 $EndComp
 $Comp
-L Device:R R?
+L Device:R R203
 U 1 1 5DD8DF60
 P 8850 5850
-F 0 "R?" H 8920 5896 50  0000 L CNN
+F 0 "R203" H 8920 5896 50  0000 L CNN
 F 1 "1k" H 8920 5805 50  0000 L CNN
-F 2 "" V 8780 5850 50  0001 C CNN
+F 2 "Resistor_SMD:R_0603_1608Metric" V 8780 5850 50  0001 C CNN
 F 3 "~" H 8850 5850 50  0001 C CNN
 	1    8850 5850
@@
 P 8500 6100
 AR Path="/5DD908F8" Ref="#PWR?"  Part="1"
-AR Path="/5DCA970B/5DD908F8" Ref="#PWR?"  Part="1"
-F 0 "#PWR?" H 8500 5850 50  0001 C CNN
+AR Path="/5DCA970B/5DD908F8" Ref="#PWR0208"  Part="1"
+F 0 "#PWR0208" H 8500 5850 50  0001 C CNN
 F 1 "GND" H 8505 5927 50  0000 C CNN
 F 2 "" H 8500 6100 50  0001 C CNN
@@
 P 8850 6100
 AR Path="/5DD90B7F" Ref="#PWR?"  Part="1"
-AR Path="/5DCA970B/5DD90B7F" Ref="#PWR?"  Part="1"
-F 0 "#PWR?" H 8850 5850 50  0001 C CNN
+AR Path="/5DCA970B/5DD90B7F" Ref="#PWR0209"  Part="1"
+F 0 "#PWR0209" H 8850 5850 50  0001 C CNN
 F 1 "GND" H 8855 5927 50  0000 C CNN
 F 2 "" H 8850 6100 50  0001 C CNN
