File: hardware/nordic_tag/dap42.sch (KiCad schematic (older format))
At the start: 16 parts

Commit message: Started PCB + BOM
Parts:
- C301, C302, C303, C304: renamed from C?; footprint (none) -> Capacitor_SMD:C_0603_1608Metric
- D301, D302, D303: renamed from D?; footprint (none) -> LED_SMD:LED_0603_1608Metric
- R301, R302, R303, R304, R305: renamed from R?; footprint (none) -> Resistor_SMD:R_0603_1608Metric
- SW301, SW302: renamed from SW?; footprint (none) -> Button_Switch_SMD:SW_Push_1P1T_NO_CK_KMR2
- Y301: renamed from Y?; footprint (none) -> Crystal:Crystal_SMD_5032-2Pin_5.0x3.2mm_HandSoldering
- gave numbers to parts that had none: 1

Commit message: Switched to pcb antenna. started placement
Parts:
- Y301: value 32MHz -> 8MHz
Changed lines of the file:
@@
 AR Path="/5DCA89B5/5DCB428B" Ref="Y301"  Part="1"
 F 0 "Y301" V 4004 2731 50  0000 L CNN
-F 1 "32MHz" V 4095 2731 50  0000 L CNN
+F 1 "8MHz" V 4095 2731 50  0000 L CNN
 F 2 "Crystal:Crystal_SMD_5032-2Pin_5.0x3.2mm_HandSoldering" H 4050 2600 50  0001 C CNN
 F 3 "~" H 4050 2600 50  0001 C CNN
